Commit message: urdf robot tophat

File: src/caramelo_description/urdf/lidar_sensor.xacro (robot description, xacro)
@@ -1,66 +1,76 @@
 <?xml version="1.0"?>
 <robot xmlns:xacro="http://www.ros.org/wiki/xacro">
-    <xacro:macro name="lidar_sensor" params="
-        prefix:=''
-        parent:='base_link'
-        frame_id:='laser_frame'
-        xyz_offset:='0 0 0'
-        rpy_offset:='0 0 0'
-        mesh_xyz_offset:='0 0 0'
-        mesh_rpy_offset:='${-M_PI/2} 0 0'
-        mesh_scale:='0.001 0.001 0.001'
-        collision_xyz_offset:='0 0 0'
-        collision_rpy_offset:='0 0 0'
-        inertial_xyz_offset:='0 0 0'
-        inertial_rpy_offset:='0 0 0'
-        lidar_width:=0.077
-        lidar_height:=0.0398
-        mass:=0.185
-        material_name:='rplidar_black'
-        material_color:='0.1 0.1 0.1 1'
-        gazebo_material_ambient:='0.1 0.1 0.1 1'
-        gazebo_material_diffuse:='0.1 0.1 0.1 1'
-        gazebo_material_specular:='0.1 0.1 0.1 1'
-        update_rate:=10
-        ray_count:=720
-        min_angle:='-3.14159'
-        max_angle:='3.14159'
-        min_range:='0.20'
-        max_range:='30.0'
-        range_resolution:='0.013'
-        topic_name:='scan'
-        always_on:=true
-        visualize:=false
-        enable_collision:=false">
-        <link name="${prefix}${frame_id}">
-        <visual>
-            <origin xyz="${mesh_xyz_offset}" rpy="${mesh_rpy_offset}"/>
-            <geometry>
-            <cylinder radius="${lidar_width/2}" length="${lidar_height}"/>
-            </geometry>
-            <material name="${material_name}">
-            <color rgba="${material_color}"/>
-            </material>
-        </visual>
-        <xacro:if value="${enable_collision}">
-            <collision>
-            <origin xyz="${collision_xyz_offset}" rpy="${collision_rpy_offset}"/>
-            <geometry>
-                <cylinder radius="${lidar_width/2}" length="${lidar_height}"/>
-            </geometry>
-            </collision>
-        </xacro:if>
-        <xacro:cylinder_inertia
-            m="${mass}"
-            r="${lidar_width/2}"
-            l="${lidar_height}"
-            o_xyz="${inertial_xyz_offset}"
-            o_rpy="${inertial_rpy_offset}"/>
-        </link>
-        <joint name="${prefix}${frame_id}_joint" type="fixed">
-        <parent link="${prefix}${parent}"/>
-        <child link="${prefix}${frame_id}" />
-        <origin xyz="${xyz_offset}" rpy="${rpy_offset}"/>
-        </joint>
-    </xacro:macro> <!-- end lidar_sensor -->
+  <xacro:property name="M_PI" value="3.1415926535897931" />
+  <xacro:macro name="lidar_sensor" params="
+    prefix:=''
+    parent:='base_link'
+    frame_id:='laser_frame'
+    mesh_file:='file://$(find caramelo_description)/urdf/meshes/rplidar_s2.stl'
+    xyz_offset:='0 0 0.0825'
+    rpy_offset:='0 0 0'
+    mesh_xyz_offset:='0 0 0'
+    mesh_rpy_offset:='${-M_PI/2} 0 0'
+    mesh_scale:='0.001 0.001 0.001'
+    collision_xyz_offset:='0 0 0'
+    collision_rpy_offset:='0 0 0'
+    inertial_xyz_offset:='0 0 0'
+    inertial_rpy_offset:='0 0 0'
+    lidar_width:=0.077
+    lidar_height:=0.0398
+    mass:=0.185
+    material_name:='rplidar_black'
+    material_color:='0.1 0.1 0.1 1'
+    gazebo_material_ambient:='0.1 0.1 0.1 1'
+    gazebo_material_diffuse:='0.1 0.1 0.1 1'
+    gazebo_material_specular:='0.1 0.1 0.1 1'
+    update_rate:=10
+    ray_count:=720
+    min_angle:='-3.14159'
+    max_angle:='3.14159'
+    min_range:='0.20'
+    max_range:='30.0'
+    range_resolution:='0.013'
+    topic_name:='/scan'
+    always_on:=true
+    visualize:=true
+    enable_collision:=false">
+    <xacro:property name="radius" value="${lidar_width/2}" />
+    <xacro:property name="ixx_iyy" value="${(mass/12) * (3 * radius * radius + lidar_height * lidar_height)}" />
+    <xacro:property name="izz" value="${(mass/2) * (radius * radius)}" />
+    <link name="${prefix}${frame_id}">
+      <visual>
+        <origin xyz="${mesh_xyz_offset}" rpy="${mesh_rpy_offset}"/>
+        <geometry>
+          <mesh filename="${mesh_file}" scale="${mesh_scale}"/>
+        </geometry>
+        <material name="${material_name}">
+          <color rgba="${material_color}"/>
+        </material>
+      </visual>
+      <xacro:if value="${enable_collision}">
+        <collision>
+          <origin xyz="${mesh_xyz_offset}" rpy="${mesh_rpy_offset}"/>
+          <geometry>
+            <mesh filename="${mesh_file}" scale="${mesh_scale}"/>
+          </geometry>
+        </collision>
+      </xacro:if>
+      <inertial>
+        <mass value="${mass}" />
+        <origin xyz="${inertial_xyz_offset}" rpy="${inertial_rpy_offset}"/>
+        <inertia
+          ixx="${ixx_iyy}"
+          ixy="0.0"
+          ixz="0.0"
+          iyy="${ixx_iyy}"
+          iyz="0.0"
+          izz="${izz}" />
+      </inertial>
+    </link>
+    <joint name="${prefix}${frame_id}_joint" type="fixed">
+      <parent link="${prefix}${parent}"/>
+      <child link="${prefix}${frame_id}" />
+      <origin xyz="${xyz_offset}" rpy="${rpy_offset}"/>
+    </joint>
+  </xacro:macro>
 </robot>

File: src/caramelo_description/urdf/mobile_base.xacro (robot description, xacro)
@@ -2,4 +2,5 @@
 <robot xmlns:xacro="http://www.ros.org/wiki/xacro">
     <xacro:include filename="mecanum_wheel.xacro"/>
+    <xacro:include filename="base_tophat.xacro"/>
     <!-- Parametros especificos do robo Caramelo -->
     <xacro:property name="base_mass" value="22.0"/>
@@ -82,4 +83,8 @@
         x_reflect="-1"
         y_reflect="-1"/>
+    <!-- Top hat on top of base -->
+    <xacro:base_tophat
+        prefix="${prefix}"
+        parent="${prefix}base_link" />
   </xacro:macro>
 </robot>

File: src/caramelo_description/urdf/robot.urdf.xacro (robot description, xacro)
@@ -11,13 +11,3 @@
   <!-- Base movel completa (base_link + footprint + 4 rodas) -->
   <xacro:mobile_base prefix="$(arg prefix)"/>
-  <!-- Sensor lidar -->
-  <xacro:lidar_sensor
-    prefix="$(arg prefix)"
-    parent="base_link"
-    frame_id="laser_frame"
-    xyz_offset="0.292 0 0.077"
-    rpy_offset="0 0 0"
-    mesh_xyz_offset="0 0 0"
-    mesh_rpy_offset="0 0 0"
-    topic_name="scan"/>
 </robot>
