Commit message: corrections

File: src/caramelo_description/urdf/base_tophat.xacro (robot description, xacro)
@@ -1,5 +1,4 @@
 <?xml version="1.0"?>
 <robot xmlns:xacro="http://www.ros.org/wiki/xacro">
-    <xacro:include filename="common_properties.xacro"/>
     <xacro:include filename="lidar_sensor.xacro"/>
     <xacro:include filename="imu.urdf.xacro"/>
@@ -22,5 +21,5 @@
                 </geometry>
                 <origin xyz="0 0 ${plate_z/2}" rpy="0 0 0"/>
-                <material name="gray"><color rgba="0.6 0.6 0.6 1.0"/></material>
+                <material name="grey"/>
             </visual>
             <collision>
@@ -42,5 +41,5 @@
                 </geometry>
                 <origin xyz="${leg_offset_x} ${leg_offset_y} ${leg_z}" rpy="0 0 0"/>
-                <material name="black"><color rgba="0.1 0.1 0.1 1.0"/></material>
+                <material name="black"/>
             </visual>
             <visual>
@@ -49,5 +48,5 @@
                 </geometry>
                 <origin xyz="${leg_offset_x} ${-leg_offset_y} ${leg_z}" rpy="0 0 0"/>
-                <material name="black"><color rgba="0.1 0.1 0.1 1.0"/></material>
+                <material name="black"/>
             </visual>
             <visual>
@@ -56,5 +55,5 @@
                 </geometry>
                 <origin xyz="${-leg_offset_x} ${leg_offset_y} ${leg_z}" rpy="0 0 0"/>
-                <material name="black"><color rgba="0.1 0.1 0.1 1.0"/></material>
+                <material name="black"/>
             </visual>
             <visual>
@@ -63,5 +62,5 @@
                 </geometry>
                 <origin xyz="${-leg_offset_x} ${-leg_offset_y} ${leg_z}" rpy="0 0 0"/>
-                <material name="black"><color rgba="0.1 0.1 0.1 1.0"/></material>
+                <material name="black"/>
             </visual>
             <collision>

File: src/caramelo_description/urdf/common_properties.xacro (robot description, xacro)
@@ -16,4 +16,7 @@
     <material name="darkgray">
         <color rgba="0.3 0.3 0.3 1.0"/>
+    </material>
+    <material name="black">
+        <color rgba="0.1 0.1 0.1 1.0"/>
     </material>
     <!-- Propriedades centrais do robo -->
