Commit message: thiago: atulização do urdf

File: src/caramelo_description/urdf/mobile_base.xacro (robot description, xacro)
@@ -2,5 +2,6 @@
 <robot xmlns:xacro="http://www.ros.org/wiki/xacro">
     <xacro:include filename="mecanum_wheel.xacro"/>
-    <xacro:include filename="base_tophat.xacro"/>
+    <xacro:include filename="lidar_sensor.xacro"/>
+    <xacro:include filename="imu.urdf.xacro"/>
     <!-- Parametros especificos do robo Caramelo -->
     <xacro:property name="base_mass" value="22.0"/>
@@ -15,34 +16,36 @@
     <xacro:property name="wheel_separation" value="0.310"/>
     <xacro:property name="wheel_base" value="0.470"/>
+    <xacro:property name="front_wheel_x" value="0.182"/>
+    <xacro:property name="back_wheel_x" value="-0.290"/>
+    <xacro:property name="left_wheel_y" value="0.145"/>
+    <xacro:property name="right_wheel_y" value="-0.145"/>
+    <xacro:property name="wheel_z" value="0.034"/>
+    <xacro:property name="base_mesh_xyz" value="-0.011611 -0.243518 -0.08"/>
+    <xacro:property name="base_mesh_rpy" value="0 0 ${M_PI/2}"/>
+    <xacro:property name="lidar_x" value="0.265"/>
+    <xacro:property name="lidar_y" value="0.000"/>
+    <xacro:property name="lidar_z" value="${base_height + 0.05 - 0.125}"/>
+    <xacro:property name="lidar_rpy" value="${M_PI} 0 ${M_PI}"/>
+    <xacro:property name="imu_x" value="-0.035"/>
+    <xacro:property name="imu_y" value="0.000"/>
+    <xacro:property name="imu_z" value="${base_height + 0.05 - 0.065}"/>
+    <xacro:property name="imu_rpy" value="0 0 0"/>
     <!-- Base completa: footprint + base_link + 4 rodas mecanum -->
     <xacro:macro name="mobile_base" params="prefix">
     <link name="${prefix}base_footprint"/>
     <link name="${prefix}base_link">
-        <!-- Corpo principal em cruz (duas caixas visuais) -->
+        <!-- Corpo principal do robo -->
         <visual>
-            <origin xyz="0 0 ${base_height/2.0}" rpy="0 0 0"/>
+            <origin xyz="${base_mesh_xyz}" rpy="${base_mesh_rpy}"/>
             <geometry>
-                <box size="${base_width_vertical} ${base_depth_vertical} ${base_height}"/>
+                <mesh filename="package://caramelo_description/urdf/meshes/montagem_robo_final.stl" scale="0.001 0.001 0.001"/>
             </geometry>
             <material name="darkgray"/>
         </visual>
-        <visual>
-            <origin xyz="0 0 ${base_height/2.0}" rpy="0 0 0"/>
+        <!-- Colisao do corpo principal -->
+        <collision>
+            <origin xyz="${base_mesh_xyz}" rpy="${base_mesh_rpy}"/>
             <geometry>
-                <box size="${base_depth_horizontal} ${base_width_horizontal} ${base_height}"/>
-            </geometry>
-            <material name="darkgray"/>
-        </visual>
-        <!-- Colisao em cruz para casar com a geometria visual -->
-        <collision>
-            <origin xyz="0 0 ${base_height/2.0}" rpy="0 0 0"/>
-            <geometry>
-                <box size="${base_width_vertical} ${base_depth_vertical} ${base_height}"/>
-            </geometry>
-        </collision>
-        <collision>
-            <origin xyz="0 0 ${base_height/2.0}" rpy="0 0 0"/>
-            <geometry>
-                <box size="${base_depth_horizontal} ${base_width_horizontal} ${base_height}"/>
+                <mesh filename="package://caramelo_description/urdf/meshes/montagem_robo_final.stl" scale="0.001 0.001 0.001"/>
             </geometry>
         </collision>
@@ -66,25 +69,33 @@
         prefix="${prefix}"
         side="front_left"
-        x_reflect="1"
-        y_reflect="1"/>
+        wheel_xyz="${front_wheel_x} ${left_wheel_y} ${wheel_z}"/>
     <xacro:mecanum_wheel
         prefix="${prefix}"
         side="front_right"
-        x_reflect="1"
-        y_reflect="-1"/>
+        wheel_xyz="${front_wheel_x} ${right_wheel_y} ${wheel_z}"
+        wheel_rpy="${-M_PI/2} 0 0"/>
     <xacro:mecanum_wheel
         prefix="${prefix}"
         side="back_left"
-        x_reflect="-1"
-        y_reflect="1"/>
+        wheel_xyz="${back_wheel_x} ${left_wheel_y} ${wheel_z}"
+        wheel_rpy="${-M_PI/2} 0 0"/>
     <xacro:mecanum_wheel
         prefix="${prefix}"
         side="back_right"
-        x_reflect="-1"
-        y_reflect="-1"/>
-    <!-- Top hat on top of base -->
-    <xacro:base_tophat
+        wheel_xyz="${back_wheel_x} ${right_wheel_y} ${wheel_z}"/>
+    <!-- Lidar no bico, preso direto na base -->
+    <xacro:lidar_sensor
         prefix="${prefix}"
-        parent="${prefix}base_link" />
+        parent="${prefix}base_link"
+        frame_id="laser_frame"
+        xyz_offset="${lidar_x} ${lidar_y} ${lidar_z}"
+        rpy_offset="${lidar_rpy}"/>
+    <!-- IMU presa direto na base -->
+    <xacro:imu_sensor
+        prefix="${prefix}"
+        parent="${prefix}base_link"
+        frame_id="imu"
+        xyz_offset="${imu_x} ${imu_y} ${imu_z}"
+        rpy_offset="${imu_rpy}"/>
   </xacro:macro>
 </robot>

File: src/manip_description/urdf/manip.ros2_control.xacro (robot description, xacro)
@@ -17,5 +17,5 @@
                 <param name="manip_joint6_motor_id">6</param>
                 <param name="manip_joint7_motor_id">7</param>
-                <param name="dynamixel_port">/dev/ttyUSB0</param>
+                <param name="dynamixel_port">/dev/ttyUSB2</param>
                 <!-- Ajuste por calibração para maior precisão de torque. -->
                 <param name="torque_constant_nm_per_amp">2.4</param>

File: urdf velho/urdf/base_tophat.xacro (robot description, xacro)
@@ -13,8 +13,4 @@
     <xacro:property name="tophat_mass" value="1.0"/>
     <xacro:property name="tophat_inertia_height" value="${plate_z + leg_height}"/>
-    <xacro:property name="lidar_x" value="0.245"/>
-    <xacro:property name="lidar_y" value="0.000"/>
-    <xacro:property name="lidar_z" value="-0.100"/>
-    <xacro:property name="lidar_rpy" value="${M_PI} 0 ${M_PI}"/>
     <!-- Macro para descrever a plataforma top hat -->
     <xacro:macro name="base_tophat" params="prefix='' parent='base_link'">
@@ -98,11 +94,11 @@
             <origin xyz="0 0 ${base_height + 0.05}" rpy="0 0 0"/>
         </joint>
-        <!-- Lidar no bico, apontado para baixo -->
+        <!-- Lidar no centro (0 0) -->
         <xacro:lidar_sensor
             prefix="${prefix}"
             parent="${prefix}base_tophat_link"
             frame_id="laser_frame"
-            xyz_offset="${lidar_x} ${lidar_y} ${lidar_z}"
-            rpy_offset="${lidar_rpy}"/>
+            xyz_offset="0 0 0.02"
+            rpy_offset="0 0 3.141592653589793"/>
         <!-- IMU em 0.10 0 -->
         <xacro:imu_sensor

File: urdf velho/urdf/mecanum_wheel.xacro (robot description, xacro)
@@ -2,19 +2,17 @@
 <robot xmlns:xacro="http://www.ros.org/wiki/xacro">
     <!-- Macro de uma roda mecanum -->
-    <xacro:macro name="mecanum_wheel" params="prefix side wheel_xyz wheel_rpy:='${M_PI/2} 0 0'">
+    <xacro:macro name="mecanum_wheel" params="prefix side x_reflect y_reflect">
         <link name="${prefix}${side}_wheel_link">
             <visual>
-                <origin xyz="0 0 0" rpy="${wheel_rpy}"/>
+                <origin xyz="0 0 0" rpy="${M_PI/2} 0 0"/>
                 <geometry>
-                    <mesh filename="package://caramelo_description/urdf/meshes/roda_escala_final.stl" scale="0.001 0.001 0.001"/>
-                    <!--<cylinder radius="${wheel_radius}" length="${wheel_width}"/>-->
+                    <cylinder radius="${wheel_radius}" length="${wheel_width}"/>
                 </geometry>
                 <material name="orange"/>
             </visual>
             <collision>
-                <origin xyz="0 0 0" rpy="${wheel_rpy}"/>
+                <origin xyz="0 0 0" rpy="${M_PI/2} 0 0"/>
                 <geometry>
-                    <mesh filename="package://caramelo_description/urdf/meshes/roda_escala_final.stl" scale="0.001 0.001 0.001"/>
-                    <!--<cylinder radius="${wheel_radius}" length="${wheel_width}"/>-->
+                    <cylinder radius="${wheel_radius}" length="${wheel_width}"/>
                 </geometry>
             </collision>
@@ -26,5 +24,5 @@
             <parent link="${prefix}base_link"/>
             <child link="${prefix}${side}_wheel_link"/>
-            <origin xyz="${wheel_xyz}" rpy="0 0 0"/>
+            <origin xyz="${x_reflect*(wheel_base/2)} ${y_reflect*(wheel_separation/2)} 0.02" rpy="0 0 0"/>
         </joint>
     </xacro:macro>
