Commit message: urdf_config

File: src/caramelo_description/urdf/control/manipulator.ros2_control.xacro (robot description, xacro)
@@ -1,13 +1,13 @@
 <?xml version="1.0"?>
 <robot xmlns:xacro="http://www.ros.org/wiki/xacro">
-    <xacro:arg name="use_mock_components" default="true"/>
+    <xacro:macro name="manipulator_ros2_control" params="use_mock_components:=true">
     <ros2_control name="Arm" type="system">
         <hardware>
-            <xacro:if value="$(arg use_mock_components)">
+            <xacro:if value="${use_mock_components}">
                 <!-- By default, set up controllers for simulation. This won't work on real hardware -->
                 <plugin>mock_components/GenericSystem</plugin>
             </xacro:if>
-            <xacro:unless value="$(arg use_mock_components)">
-                <plugin>arm_hardware/ArmHardwareInterface</plugin>
+            <xacro:unless value="${use_mock_components}">
+                <plugin>arm_hardware_interface/ArmHWInterface</plugin>
                 <param name="manip_joint1_motor_id">1</param>
                 <param name="manip_joint2_motor_id">2</param>
@@ -93,3 +93,4 @@
         </joint>
     </ros2_control>
+    </xacro:macro>
 </robot>

File: src/caramelo_description/urdf/mech/base_tophat.xacro (robot description, xacro)
@@ -1,6 +1,6 @@
 <?xml version="1.0"?>
 <robot xmlns:xacro="http://www.ros.org/wiki/xacro">
-    <xacro:include filename="lidar_sensor.xacro"/>
-    <xacro:include filename="imu.urdf.xacro"/>
+    <xacro:include filename="../sensors/lidar_sensor.xacro"/>
+    <xacro:include filename="../sensors/imu.urdf.xacro"/>
     <xacro:property name="plate_x" value="0.315"/>
     <xacro:property name="plate_y" value="0.30"/>

File: src/caramelo_description/urdf/mech/manipulator_arm.xacro (robot description, xacro)
@@ -1,14 +1,11 @@
 <?xml version="1.0"?>
 <robot name="manip" xmlns:xacro="http://ros.org/wiki/xacro">
-  <!-- ================= REALSENSE INCLUDE ================= -->
-  <xacro:arg name="use_realsense" default="true"/>
-  <xacro:if value="$(arg use_realsense)">
-    <xacro:include filename="$(find realsense2_description)/urdf/_d455.urdf.xacro"/>
-  </xacro:if>
+  <xacro:include filename="../sensors/rgbd_camera.urdf.xacro"/>
+  <xacro:macro name="manip_arm" params="base_link_name:='base_link' use_realsense:=true">
   <!-- ================= BASE ================= -->
-  <link name="base_link">
-    <visual>
-      <geometry>
-        <mesh filename="package://manip_description/meshes/base_link.stl" scale="0.001 0.001 0.001"/>
+  <link name="${base_link_name}">
+    <visual>
+      <geometry>
+        <mesh filename="package://caramelo_description/meshes/manipulator/base_link.stl" scale="0.001 0.001 0.001"/>
       </geometry>
       <origin xyz="0 0 0" rpy="0 0 0"/>
@@ -16,5 +13,5 @@
     <collision>
       <geometry>
-        <mesh filename="package://manip_description/meshes/base_link.stl" scale="0.001 0.001 0.001"/>
+        <mesh filename="package://caramelo_description/meshes/manipulator/base_link.stl" scale="0.001 0.001 0.001"/>
       </geometry>
       <origin xyz="0 0 0" rpy="0 0 0"/>
@@ -32,5 +29,5 @@
     <visual>
       <geometry>
-        <mesh filename="package://manip_description/meshes/link1.stl" scale="0.001 0.001 0.001"/>
+        <mesh filename="package://caramelo_description/meshes/manipulator/link1.stl" scale="0.001 0.001 0.001"/>
       </geometry>
       <origin xyz="0 0 0.0" rpy="0 0 0"/>
@@ -41,5 +38,5 @@
     <collision>
       <geometry>
-        <mesh filename="package://manip_description/meshes/link1.stl" scale="0.001 0.001 0.001"/>
+        <mesh filename="package://caramelo_description/meshes/manipulator/link1.stl" scale="0.001 0.001 0.001"/>
       </geometry>
       <origin xyz="0 0 0.0" rpy="0 0 0"/>
@@ -57,5 +54,5 @@
     <visual>
       <geometry>
-        <mesh filename="package://manip_description/meshes/link2.stl" scale="0.001 0.001 0.001"/>
+        <mesh filename="package://caramelo_description/meshes/manipulator/link2.stl" scale="0.001 0.001 0.001"/>
       </geometry>
       <origin xyz="0 0 -0.09775" rpy="0 0 0"/>
@@ -66,5 +63,5 @@
     <collision>
       <geometry>
-        <mesh filename="package://manip_description/meshes/link2.stl" scale="0.001 0.001 0.001"/>
+        <mesh filename="package://caramelo_description/meshes/manipulator/link2.stl" scale="0.001 0.001 0.001"/>
       </geometry>
       <origin xyz="0 0 -0.09775" rpy="0 0 0"/>
@@ -82,5 +79,5 @@
     <visual>
       <geometry>
-        <mesh filename="package://manip_description/meshes/link3.stl" scale="0.001 0.001 0.001"/>
+        <mesh filename="package://caramelo_description/meshes/manipulator/link3.stl" scale="0.001 0.001 0.001"/>
       </geometry>
       <origin xyz="0 0 -0.28275" rpy="0 0 0"/>
@@ -91,5 +88,5 @@
     <collision>
       <geometry>
-        <mesh filename="package://manip_description/meshes/link3.stl" scale="0.001 0.001 0.001"/>
+        <mesh filename="package://caramelo_description/meshes/manipulator/link3.stl" scale="0.001 0.001 0.001"/>
       </geometry>
       <origin xyz="0 0 -0.28275" rpy="0 0 0"/>
@@ -107,5 +104,5 @@
     <visual>
       <geometry>
-        <mesh filename="package://manip_description/meshes/link4.stl" scale="0.001 0.001 0.001"/>
+        <mesh filename="package://caramelo_description/meshes/manipulator/link4.stl" scale="0.001 0.001 0.001"/>
       </geometry>
       <origin xyz="0 0 -0.48775" rpy="0 0 3.14"/>
@@ -116,5 +113,5 @@
     <collision>
       <geometry>
-        <mesh filename="package://manip_description/meshes/link4.stl" scale="0.001 0.001 0.001"/>
+        <mesh filename="package://caramelo_description/meshes/manipulator/link4.stl" scale="0.001 0.001 0.001"/>
       </geometry>
       <origin xyz="0 0 -0.48775" rpy="0 0 0"/>
@@ -132,5 +129,5 @@
     <visual>
       <geometry>
-        <mesh filename="package://manip_description/meshes/link5.stl" scale="0.001 0.001 0.001"/>
+        <mesh filename="package://caramelo_description/meshes/manipulator/link5.stl" scale="0.001 0.001 0.001"/>
       </geometry>
       <origin xyz="0 0 -0.5659" rpy="0.0 0 0"/>
@@ -141,5 +138,5 @@
     <collision>
       <geometry>
-        <mesh filename="package://manip_description/meshes/link5.stl" scale="0.001 0.001 0.001"/>
+        <mesh filename="package://caramelo_description/meshes/manipulator/link5.stl" scale="0.001 0.001 0.001"/>
       </geometry>
       <origin xyz="0 0 -0.5659" rpy="0.0 0 0"/>
@@ -154,19 +151,15 @@
   </link>
   <!-- ================= REALSENSE D455 ================= -->
-  <xacro:if value="$(arg use_realsense)">
-    <xacro:sensor_d455
+  <xacro:if value="${use_realsense}">
+    <xacro:rgbd_camera
         parent="link5"
-        name="camera"
-        use_nominal_extrinsics="true">
-        <!--
-        Ajuste da pose da câmera em relação ao flange
-        -->
-        <origin xyz="0 -0.055 0.0125"
-                rpy="0 -1.57079632679 -1.57079632679"/>
-    </xacro:sensor_d455>
+        camera_name="camera"
+        use_nominal_extrinsics="true"
+        xyz_offset="0 -0.055 0.0125"
+        rpy_offset="0 -1.57079632679 -1.57079632679"/>
   </xacro:if>
   <!-- ================= ARM JOINTS ================= -->
   <joint name="manip_joint1" type="revolute">
-    <parent link="base_link"/>
+    <parent link="${base_link_name}"/>
     <child link="link1"/>
     <axis xyz="0 0 1"/>
@@ -236,3 +229,4 @@
     <origin xyz="0 0 0.3" rpy="0 0 0"/>
   </joint>
+  </xacro:macro>
 </robot>

File: src/caramelo_description/urdf/mech/manipulator_gripper.xacro (robot description, xacro)
@@ -1,4 +1,5 @@
 <?xml version="1.0"?>
 <robot xmlns:xacro="http://www.ros.org/wiki/xacro">
+    <xacro:macro name="manip_gripper">
     <link name="gripper_base_link">
     <visual>
@@ -15,5 +16,5 @@
     <visual>
         <geometry>
-        <mesh filename="package://manip_description/meshes/left_finger.stl" scale="0.001 0.001 0.001"/>
+        <mesh filename="package://caramelo_description/meshes/manipulator/left_finger.stl" scale="0.001 0.001 0.001"/>
         </geometry>
         <origin xyz="-0.0252 0 -0.58444" rpy="0 0 0"/>
@@ -24,5 +25,5 @@
     <collision>
         <geometry>
-        <mesh filename="package://manip_description/meshes/left_finger.stl" scale="0.001 0.001 0.001"/>
+        <mesh filename="package://caramelo_description/meshes/manipulator/left_finger.stl" scale="0.001 0.001 0.001"/>
         </geometry>
         <origin xyz="-0.0252 0 -0.58444" rpy="0 0 0"/>
@@ -44,5 +45,5 @@
     <visual>
         <geometry>
-        <mesh filename="package://manip_description/meshes/right_finger.stl" scale="0.001 0.001 0.001"/>
+        <mesh filename="package://caramelo_description/meshes/manipulator/right_finger.stl" scale="0.001 0.001 0.001"/>
         </geometry>
         <origin xyz="0.0252 0 -0.58444" rpy="0 0 0"/>
@@ -51,5 +52,5 @@
     <collision>
         <geometry>
-        <mesh filename="package://manip_description/meshes/right_finger.stl" scale="0.001 0.001 0.001"/>
+        <mesh filename="package://caramelo_description/meshes/manipulator/right_finger.stl" scale="0.001 0.001 0.001"/>
         </geometry>
         <origin xyz="0.0252 0 -0.58444" rpy="0 0 0"/>
@@ -68,3 +69,4 @@
     <limit lower="-1.0" upper="1.0" effort="1" velocity="5"/>
     </joint>
+    </xacro:macro>
 </robot>

File: src/caramelo_description/urdf/mech/mecanum_wheel.xacro (robot description, xacro)
@@ -1,30 +1,36 @@
 <?xml version="1.0"?>
 <robot xmlns:xacro="http://www.ros.org/wiki/xacro">
-    <!-- Macro de uma roda mecanum -->
-    <xacro:macro name="mecanum_wheel" params="prefix side wheel_xyz wheel_rpy:='${M_PI/2} 0 0'">
+    <xacro:property name="mecanum_wheel_mesh" value="package://caramelo_description/meshes/robot_3d/roda_escala_final.stl"/>
+    <xacro:property name="mecanum_wheel_mesh_scale" value="0.001 0.001 0.001"/>
+    <!-- ROS2_CONTROL: os nomes das juntas sao contrato com caramelo_controllers.yaml e mobile_base_hw_interface.cpp. -->
+    <xacro:macro name="mecanum_wheel" params="
+        prefix
+        side
+        x_reflect
+        y_reflect
+        wheel_mesh:='${mecanum_wheel_mesh}'
+        wheel_mesh_scale:='${mecanum_wheel_mesh_scale}'">
         <link name="${prefix}${side}_wheel_link">
             <visual>
-                <origin xyz="0 0 0" rpy="${wheel_rpy}"/>
+                <origin xyz="0 0 0" rpy="${M_PI/2 if x_reflect == y_reflect else -M_PI/2} 0 0"/>
                 <geometry>
-                    <mesh filename="package://caramelo_description/urdf/meshes/roda_escala_final.stl" scale="0.001 0.001 0.001"/>
-                    <!--<cylinder radius="${wheel_radius}" length="${wheel_width}"/>-->
+                    <mesh filename="${wheel_mesh}" scale="${wheel_mesh_scale}"/>
                 </geometry>
                 <material name="orange"/>
             </visual>
             <collision>
-                <origin xyz="0 0 0" rpy="${wheel_rpy}"/>
+                <origin xyz="0 0 0" rpy="${M_PI/2 if x_reflect == y_reflect else -M_PI/2} 0 0"/>
                 <geometry>
-                    <mesh filename="package://caramelo_description/urdf/meshes/roda_escala_final.stl" scale="0.001 0.001 0.001"/>
-                    <!--<cylinder radius="${wheel_radius}" length="${wheel_width}"/>-->
+                    <mesh filename="${wheel_mesh}" scale="${wheel_mesh_scale}"/>
                 </geometry>
             </collision>
             <xacro:cylinder_inertia m="${wheel_mass}" r="${wheel_radius}" l="${wheel_width}" o_xyz="0 0 0" o_rpy="${M_PI/2} 0 0"/>
         </link>
-        <!-- Rotacao continua da roda no eixo Y -->
+        <!-- FRAME_CRITICO: rotacao continua da roda no eixo Y. -->
         <joint name="${prefix}${side}_wheel_joint" type="continuous">
             <axis xyz="0 1 0"/>
             <parent link="${prefix}base_link"/>
             <child link="${prefix}${side}_wheel_link"/>
-            <origin xyz="${wheel_xyz}" rpy="0 0 0"/>
+            <origin xyz="${wheel_center_x + x_reflect*(wheel_base/2)} ${y_reflect*(wheel_separation/2)} ${wheel_z}" rpy="0 0 0"/>
         </joint>
     </xacro:macro>

File: src/caramelo_description/urdf/mech/mobile_base.xacro (robot description, xacro)
@@ -2,32 +2,42 @@
 <robot xmlns:xacro="http://www.ros.org/wiki/xacro">
     <xacro:include filename="mecanum_wheel.xacro"/>
-    <xacro:include filename="lidar_sensor.xacro"/>
-    <xacro:include filename="imu.urdf.xacro"/>
+    <xacro:include filename="../sensors/lidar_sensor.xacro"/>
+    <xacro:include filename="../sensors/imu.urdf.xacro"/>
     <!-- Parametros especificos do robo Caramelo -->
     <xacro:property name="base_mass" value="22.0"/>
-    <xacro:property name="base_height" value="0.105"/>
-    <xacro:property name="base_width_vertical" value="0.550"/>
+    <!-- Medidas do chassi sem considerar o apendice frontal do LiDAR. -->
+    <xacro:property name="base_height" value="0.156"/>
+    <xacro:property name="base_width_vertical" value="0.535"/>
     <xacro:property name="base_depth_vertical" value="0.210"/>
-    <xacro:property name="base_width_horizontal" value="0.330"/>
+    <xacro:property name="base_width_horizontal" value="0.316"/>
     <xacro:property name="base_depth_horizontal" value="0.320"/>
+    <xacro:property name="chassis_bottom_from_floor" value="0.018"/>
+    <xacro:property name="base_link_z_from_floor" value="${chassis_bottom_from_floor + base_height/2.0}"/>
+    <xacro:property name="base_appendage_x" value="0.108"/>
+    <!-- Referencia antiga usada para manter sensores na mesma altura absoluta apos mover o base_link. -->
+    <xacro:property name="old_base_link_z_from_floor" value="0.030"/>
     <xacro:property name="wheel_radius" value="0.05"/>
     <xacro:property name="wheel_width" value="0.069"/>
     <xacro:property name="wheel_mass" value="3.0"/>
-    <xacro:property name="wheel_separation" value="0.310"/>
-    <xacro:property name="wheel_base" value="0.470"/>
-    <xacro:property name="front_wheel_x" value="0.182"/>
-    <xacro:property name="back_wheel_x" value="-0.290"/>
-    <xacro:property name="left_wheel_y" value="0.145"/>
-    <xacro:property name="right_wheel_y" value="-0.145"/>
-    <xacro:property name="wheel_z" value="0.034"/>
-    <xacro:property name="base_mesh_xyz" value="-0.011611 -0.243518 -0.08"/>
+    <!-- AJUSTAR_NO_ROBO: conferir posicao real das rodas e offset do STL no robo montado. -->
+    <xacro:property name="wheel_separation" value="0.290"/>
+    <xacro:property name="wheel_base" value="0.472"/>
+    <xacro:property name="wheel_center_x" value="0.000"/>
+    <xacro:property name="wheel_z" value="${wheel_radius - base_link_z_from_floor}"/>
+    <!-- FRAME_CRITICO: offsets medidos do STL ja com a rotacao de 90 graus aplicada abaixo. -->
+    <xacro:property name="base_mesh_stl_center_x" value="0.243517868"/>
+    <xacro:property name="base_mesh_stl_center_y" value="-0.011611206"/>
+    <xacro:property name="base_mesh_stl_min_z" value="0.080840126"/>
+    <xacro:property name="base_mesh_xyz" value="${base_appendage_x/2.0 + base_mesh_stl_center_y} ${-base_mesh_stl_center_x} ${-(base_height/2.0 + base_mesh_stl_min_z)}"/>
     <xacro:property name="base_mesh_rpy" value="0 0 ${M_PI/2}"/>
-    <xacro:property name="lidar_x" value="0.265"/>
+    <!-- FRAME_CRITICO: manter o frame publicado pelo driver do LiDAR igual ao rplidar_s2.yaml. -->
+    <xacro:property name="lidar_x" value="${0.265 + base_appendage_x/2.0}"/>
     <xacro:property name="lidar_y" value="0.000"/>
-    <xacro:property name="lidar_z" value="${base_height + 0.05 - 0.125}"/>
+    <xacro:property name="lidar_z" value="${old_base_link_z_from_floor + 0.030 - base_link_z_from_floor}"/>
     <xacro:property name="lidar_rpy" value="${M_PI} 0 ${M_PI}"/>
-    <xacro:property name="imu_x" value="-0.035"/>
+    <!-- FRAME_CRITICO: hardware_bringup publica a IMU como imu_link. -->
+    <xacro:property name="imu_x" value="${-0.035 + base_appendage_x/2.0}"/>
     <xacro:property name="imu_y" value="0.000"/>
-    <xacro:property name="imu_z" value="${base_height + 0.05 - 0.065}"/>
+    <xacro:property name="imu_z" value="${old_base_link_z_from_floor + 0.090 - base_link_z_from_floor}"/>
     <xacro:property name="imu_rpy" value="0 0 0"/>
     <!-- Base completa: footprint + base_link + 4 rodas mecanum -->
@@ -39,5 +49,5 @@
             <origin xyz="${base_mesh_xyz}" rpy="${base_mesh_rpy}"/>
             <geometry>
-                <mesh filename="package://caramelo_description/urdf/meshes/montagem_robo_final.stl" scale="0.001 0.001 0.001"/>
+                <mesh filename="package://caramelo_description/meshes/robot_3d/montagem_robo_final.stl" scale="0.001 0.001 0.001"/>
             </geometry>
             <material name="darkgray"/>
@@ -47,5 +57,5 @@
             <origin xyz="${base_mesh_xyz}" rpy="${base_mesh_rpy}"/>
             <geometry>
-                <mesh filename="package://caramelo_description/urdf/meshes/montagem_robo_final.stl" scale="0.001 0.001 0.001"/>
+                <mesh filename="package://caramelo_description/meshes/robot_3d/montagem_robo_final.stl" scale="0.001 0.001 0.001"/>
             </geometry>
         </collision>
@@ -56,5 +66,5 @@
             y="${base_width_horizontal}"
             z="${base_height}"
-            o_xyz="0 0 ${base_height/2.0}"
+            o_xyz="0 0 0"
             o_rpy="0 0 0"/>
     </link>
@@ -63,5 +73,5 @@
         <parent link="${prefix}base_footprint"/>
         <child link="${prefix}base_link"/>
-        <origin xyz="0 0 ${wheel_radius - 0.02}" rpy="0 0 0"/>
+        <origin xyz="0 0 ${base_link_z_from_floor}" rpy="0 0 0"/>
     </joint>
     <!-- Quatro rodas mecanum -->
@@ -69,19 +79,21 @@
         prefix="${prefix}"
         side="front_left"
-        wheel_xyz="${front_wheel_x} ${left_wheel_y} ${wheel_z}"/>
+        x_reflect="1"
+        y_reflect="1"/>
     <xacro:mecanum_wheel
         prefix="${prefix}"
         side="front_right"
-        wheel_xyz="${front_wheel_x} ${right_wheel_y} ${wheel_z}"
-        wheel_rpy="${-M_PI/2} 0 0"/>
+        x_reflect="1"
+        y_reflect="-1"/>
     <xacro:mecanum_wheel
         prefix="${prefix}"
         side="back_left"
-        wheel_xyz="${back_wheel_x} ${left_wheel_y} ${wheel_z}"
-        wheel_rpy="${-M_PI/2} 0 0"/>
+        x_reflect="-1"
+        y_reflect="1"/>
     <xacro:mecanum_wheel
         prefix="${prefix}"
         side="back_right"
-        wheel_xyz="${back_wheel_x} ${right_wheel_y} ${wheel_z}"/>
+        x_reflect="-1"
+        y_reflect="-1"/>
     <!-- Lidar no bico, preso direto na base -->
     <xacro:lidar_sensor

File: src/caramelo_description/urdf/robots/robot.urdf.xacro (robot description, xacro)
@@ -4,10 +4,25 @@
   <xacro:arg name="robot_name" default="caramelo"/>
   <xacro:arg name="prefix" default=""/>
+  <xacro:arg name="use_manipulator" default="true"/>
+  <xacro:arg name="use_realsense" default="true"/>
+  <xacro:arg name="use_mock_components" default="true"/>
+  <xacro:arg name="manip_mount_xyz" default="0.185 0 0.078"/>
+  <xacro:arg name="manip_mount_rpy" default="0 0 0"/>
   <!-- Includes -->
-  <xacro:include filename="common_properties.xacro"/>
-  <xacro:include filename="lidar_sensor.xacro"/>
-  <xacro:include filename="mobile_base.xacro"/>
-  <xacro:include filename="mobile_base.ros2_control.xacro"/>
+  <xacro:include filename="../materials.xacro"/>
+  <xacro:include filename="../mech/mobile_base.xacro"/>
+  <xacro:include filename="../control/mobile_base.ros2_control.xacro"/>
+  <xacro:include filename="../control/manipulator.ros2_control.xacro"/>
+  <xacro:include filename="../mech/caramelo_manipulator.xacro"/>
   <!-- Base movel completa (base_link + footprint + 4 rodas) -->
   <xacro:mobile_base prefix="$(arg prefix)"/>
+  <xacro:if value="$(arg use_manipulator)">
+    <xacro:caramelo_manipulator
+      prefix="$(arg prefix)"
+      parent="$(arg prefix)base_link"
+      use_realsense="$(arg use_realsense)"
+      manip_mount_xyz="$(arg manip_mount_xyz)"
+      manip_mount_rpy="$(arg manip_mount_rpy)"/>
+    <xacro:manipulator_ros2_control use_mock_components="$(arg use_mock_components)"/>
+  </xacro:if>
 </robot>

File: src/caramelo_description/urdf/sensors/lidar_sensor.xacro (robot description, xacro)
@@ -6,5 +6,5 @@
     parent:='base_link'
     frame_id:='laser_frame'
-    mesh_file:='file://$(find caramelo_description)/urdf/meshes/rplidar_s2.stl'
+    mesh_file:='package://caramelo_description/meshes/rplidar/rplidar_s2.stl'
     xyz_offset:='0 0 0.0825'
     rpy_offset:='0 0 0'
