Commit message: Refactor robot description and launch configurations
- Updated mobile_base.xacro to support visual modes and mesh URI prefixes.
- Modified manipulator.urdf.xacro and robot.urdf.xacro to include visual mode and mesh URI arguments.
- Enhanced lidar_sensor.xacro to allow for visual mode selection.
- Adjusted caramelo_controllers.yaml to include arm and gripper controllers with updated parameters.
- Removed obsolete manip_ros2_controllers.yaml and consolidated configurations into caramelo_controllers.yaml.
- Updated rplidar_s2.yaml to change serial port and scan mode.
- Added USB rules for stable device naming on Raspberry Pi.
- Introduced scan_normalizer.yaml and scan_normalizer.py for processing LaserScan messages.
- Cleaned up unused launch files related to manipulator control.
- Added rviz_remote.launch.py for remote RViz configuration.

File: src/caramelo_description/urdf/control/manipulator.ros2_control.xacro (robot description, xacro)
@@ -17,5 +17,5 @@
                 <param name="manip_joint6_motor_id">6</param>
                 <param name="manip_joint7_motor_id">7</param>
-                <param name="dynamixel_port">/dev/ttyUSB2</param>
+                <param name="dynamixel_port">/dev/manip_usb</param>
                 <!-- Ajuste por calibração para maior precisão de torque. -->
                 <param name="torque_constant_nm_per_amp">2.4</param>

File: src/caramelo_description/urdf/mech/caramelo_manipulator.xacro (robot description, xacro)
@@ -7,6 +7,8 @@
     parent:='base_link'
     use_realsense:=true
-    manip_mount_xyz:='0.185 0 0.078'
-    manip_mount_rpy:='0 0 0'">
+    manip_mount_xyz:='0.217 0 0.083'
+    manip_mount_rpy:='0 0 0'
+    visual_mode:='package'
+    mesh_uri_prefix:='package://caramelo_description'">
     <!-- AJUSTAR_NO_ROBO: conferir a pose real do suporte do manipulador no chassi. -->
     <joint name="${prefix}manipulator_mount_joint" type="fixed">
@@ -16,6 +18,12 @@
     </joint>
     <!-- IMPORTANTE: o base_link do manipulador vira manip_base_link para nao colidir com a base movel. -->
-    <xacro:manip_arm base_link_name="manip_base_link" use_realsense="${use_realsense}"/>
-    <xacro:manip_gripper/>
+    <xacro:manip_arm
+      base_link_name="manip_base_link"
+      use_realsense="${use_realsense}"
+      visual_mode="${visual_mode}"
+      mesh_uri_prefix="${mesh_uri_prefix}"/>
+    <xacro:manip_gripper
+      visual_mode="${visual_mode}"
+      mesh_uri_prefix="${mesh_uri_prefix}"/>
     <joint name="${prefix}gripper_base_joint" type="fixed">
       <parent link="link5"/>

File: src/caramelo_description/urdf/mech/manipulator_arm.xacro (robot description, xacro)
@@ -2,10 +2,19 @@
 <robot name="manip" xmlns:xacro="http://ros.org/wiki/xacro">
   <xacro:include filename="../sensors/rgbd_camera.urdf.xacro"/>
-  <xacro:macro name="manip_arm" params="base_link_name:='base_link' use_realsense:=true">
+  <xacro:macro name="manip_arm" params="
+    base_link_name:='base_link'
+    use_realsense:=true
+    visual_mode:='package'
+    mesh_uri_prefix:='package://caramelo_description'">
   <!-- ================= BASE ================= -->
   <link name="${base_link_name}">
     <visual>
       <geometry>
-        <mesh filename="package://caramelo_description/meshes/manipulator/base_link.stl" scale="0.001 0.001 0.001"/>
+        <xacro:if value="${visual_mode == 'primitive'}">
+          <cylinder radius="0.065" length="0.055"/>
+        </xacro:if>
+        <xacro:if value="${visual_mode != 'primitive'}">
+          <mesh filename="${mesh_uri_prefix}/meshes/manipulator/base_link.stl" scale="0.001 0.001 0.001"/>
+        </xacro:if>
       </geometry>
       <origin xyz="0 0 0" rpy="0 0 0"/>
@@ -13,5 +22,10 @@
     <collision>
       <geometry>
-        <mesh filename="package://caramelo_description/meshes/manipulator/base_link.stl" scale="0.001 0.001 0.001"/>
+        <xacro:if value="${visual_mode == 'primitive'}">
+          <cylinder radius="0.065" length="0.055"/>
+        </xacro:if>
+        <xacro:if value="${visual_mode != 'primitive'}">
+          <mesh filename="${mesh_uri_prefix}/meshes/manipulator/base_link.stl" scale="0.001 0.001 0.001"/>
+        </xacro:if>
       </geometry>
       <origin xyz="0 0 0" rpy="0 0 0"/>
@@ -29,5 +43,10 @@
     <visual>
       <geometry>
-        <mesh filename="package://caramelo_description/meshes/manipulator/link1.stl" scale="0.001 0.001 0.001"/>
+        <xacro:if value="${visual_mode == 'primitive'}">
+          <cylinder radius="0.045" length="0.100"/>
+        </xacro:if>
+        <xacro:if value="${visual_mode != 'primitive'}">
+          <mesh filename="${mesh_uri_prefix}/meshes/manipulator/link1.stl" scale="0.001 0.001 0.001"/>
+        </xacro:if>
       </geometry>
       <origin xyz="0 0 0.0" rpy="0 0 0"/>
@@ -38,5 +57,10 @@
     <collision>
       <geometry>
-        <mesh filename="package://caramelo_description/meshes/manipulator/link1.stl" scale="0.001 0.001 0.001"/>
+        <xacro:if value="${visual_mode == 'primitive'}">
+          <cylinder radius="0.045" length="0.100"/>
+        </xacro:if>
+        <xacro:if value="${visual_mode != 'primitive'}">
+          <mesh filename="${mesh_uri_prefix}/meshes/manipulator/link1.stl" scale="0.001 0.001 0.001"/>
+        </xacro:if>
       </geometry>
       <origin xyz="0 0 0.0" rpy="0 0 0"/>
@@ -54,5 +78,10 @@
     <visual>
       <geometry>
-        <mesh filename="package://caramelo_description/meshes/manipulator/link2.stl" scale="0.001 0.001 0.001"/>
+        <xacro:if value="${visual_mode == 'primitive'}">
+          <box size="0.055 0.055 0.185"/>
+        </xacro:if>
+        <xacro:if value="${visual_mode != 'primitive'}">
+          <mesh filename="${mesh_uri_prefix}/meshes/manipulator/link2.stl" scale="0.001 0.001 0.001"/>
+        </xacro:if>
       </geometry>
       <origin xyz="0 0 -0.09775" rpy="0 0 0"/>
@@ -63,5 +92,10 @@
     <collision>
       <geometry>
-        <mesh filename="package://caramelo_description/meshes/manipulator/link2.stl" scale="0.001 0.001 0.001"/>
+        <xacro:if value="${visual_mode == 'primitive'}">
+          <box size="0.055 0.055 0.185"/>
+        </xacro:if>
+        <xacro:if value="${visual_mode != 'primitive'}">
+          <mesh filename="${mesh_uri_prefix}/meshes/manipulator/link2.stl" scale="0.001 0.001 0.001"/>
+        </xacro:if>
       </geometry>
       <origin xyz="0 0 -0.09775" rpy="0 0 0"/>
@@ -79,5 +113,10 @@
     <visual>
       <geometry>
-        <mesh filename="package://caramelo_description/meshes/manipulator/link3.stl" scale="0.001 0.001 0.001"/>
+        <xacro:if value="${visual_mode == 'primitive'}">
+          <box size="0.050 0.050 0.205"/>
+        </xacro:if>
+        <xacro:if value="${visual_mode != 'primitive'}">
+          <mesh filename="${mesh_uri_prefix}/meshes/manipulator/link3.stl" scale="0.001 0.001 0.001"/>
+        </xacro:if>
       </geometry>
       <origin xyz="0 0 -0.28275" rpy="0 0 0"/>
@@ -88,5 +127,10 @@
     <collision>
       <geometry>
-        <mesh filename="package://caramelo_description/meshes/manipulator/link3.stl" scale="0.001 0.001 0.001"/>
+        <xacro:if value="${visual_mode == 'primitive'}">
+          <box size="0.050 0.050 0.205"/>
+        </xacro:if>
+        <xacro:if value="${visual_mode != 'primitive'}">
+          <mesh filename="${mesh_uri_prefix}/meshes/manipulator/link3.stl" scale="0.001 0.001 0.001"/>
+        </xacro:if>
       </geometry>
       <origin xyz="0 0 -0.28275" rpy="0 0 0"/>
@@ -104,5 +148,10 @@
     <visual>
       <geometry>
-        <mesh filename="package://caramelo_description/meshes/manipulator/link4.stl" scale="0.001 0.001 0.001"/>
+        <xacro:if value="${visual_mode == 'primitive'}">
+          <box size="0.050 0.050 0.160"/>
+        </xacro:if>
+        <xacro:if value="${visual_mode != 'primitive'}">
+          <mesh filename="${mesh_uri_prefix}/meshes/manipulator/link4.stl" scale="0.001 0.001 0.001"/>
+        </xacro:if>
       </geometry>
       <origin xyz="0 0 -0.48775" rpy="0 0 3.14"/>
@@ -113,5 +162,10 @@
     <collision>
       <geometry>
-        <mesh filename="package://caramelo_description/meshes/manipulator/link4.stl" scale="0.001 0.001 0.001"/>
+        <xacro:if value="${visual_mode == 'primitive'}">
+          <box size="0.050 0.050 0.160"/>
+        </xacro:if>
+        <xacro:if value="${visual_mode != 'primitive'}">
+          <mesh filename="${mesh_uri_prefix}/meshes/manipulator/link4.stl" scale="0.001 0.001 0.001"/>
+        </xacro:if>
       </geometry>
       <origin xyz="0 0 -0.48775" rpy="0 0 0"/>
@@ -129,5 +183,10 @@
     <visual>
       <geometry>
-        <mesh filename="package://caramelo_description/meshes/manipulator/link5.stl" scale="0.001 0.001 0.001"/>
+        <xacro:if value="${visual_mode == 'primitive'}">
+          <cylinder radius="0.035" length="0.080"/>
+        </xacro:if>
+        <xacro:if value="${visual_mode != 'primitive'}">
+          <mesh filename="${mesh_uri_prefix}/meshes/manipulator/link5.stl" scale="0.001 0.001 0.001"/>
+        </xacro:if>
       </geometry>
       <origin xyz="0 0 -0.5659" rpy="0.0 0 0"/>
@@ -138,5 +197,10 @@
     <collision>
       <geometry>
-        <mesh filename="package://caramelo_description/meshes/manipulator/link5.stl" scale="0.001 0.001 0.001"/>
+        <xacro:if value="${visual_mode == 'primitive'}">
+          <cylinder radius="0.035" length="0.080"/>
+        </xacro:if>
+        <xacro:if value="${visual_mode != 'primitive'}">
+          <mesh filename="${mesh_uri_prefix}/meshes/manipulator/link5.stl" scale="0.001 0.001 0.001"/>
+        </xacro:if>
       </geometry>
       <origin xyz="0 0 -0.5659" rpy="0.0 0 0"/>
@@ -156,4 +220,6 @@
         camera_name="camera"
         use_nominal_extrinsics="true"
+        visual_mode="${visual_mode}"
+        mesh_uri_prefix="${mesh_uri_prefix}"
         xyz_offset="0 -0.055 0.0125"
         rpy_offset="0 -1.57079632679 -1.57079632679"/>

File: src/caramelo_description/urdf/mech/manipulator_gripper.xacro (robot description, xacro)
@@ -1,5 +1,7 @@
 <?xml version="1.0"?>
 <robot xmlns:xacro="http://www.ros.org/wiki/xacro">
-    <xacro:macro name="manip_gripper">
+    <xacro:macro name="manip_gripper" params="
+        visual_mode:='package'
+        mesh_uri_prefix:='package://caramelo_description'">
     <link name="gripper_base_link">
     <visual>
@@ -16,7 +18,12 @@
     <visual>
         <geometry>
-        <mesh filename="package://caramelo_description/meshes/manipulator/left_finger.stl" scale="0.001 0.001 0.001"/>
+        <xacro:if value="${visual_mode == 'primitive'}">
+        <box size="0.018 0.018 0.090"/>
+        </xacro:if>
+        <xacro:if value="${visual_mode != 'primitive'}">
+        <mesh filename="${mesh_uri_prefix}/meshes/manipulator/left_finger.stl" scale="0.001 0.001 0.001"/>
+        </xacro:if>
         </geometry>
-        <origin xyz="-0.0252 0 -0.58444" rpy="0 0 0"/>
+        <origin xyz="${0 if visual_mode == 'primitive' else -0.0252} 0 ${-0.045 if visual_mode == 'primitive' else -0.58444}" rpy="0 0 0"/>
         <material name="grey">
         <color rgba="0.6 0.6 0.6 1"/>
@@ -25,7 +32,12 @@
     <collision>
         <geometry>
-        <mesh filename="package://caramelo_description/meshes/manipulator/left_finger.stl" scale="0.001 0.001 0.001"/>
+        <xacro:if value="${visual_mode == 'primitive'}">
+        <box size="0.018 0.018 0.090"/>
+        </xacro:if>
+        <xacro:if value="${visual_mode != 'primitive'}">
+        <mesh filename="${mesh_uri_prefix}/meshes/manipulator/left_finger.stl" scale="0.001 0.001 0.001"/>
+        </xacro:if>
         </geometry>
-        <origin xyz="-0.0252 0 -0.58444" rpy="0 0 0"/>
+        <origin xyz="${0 if visual_mode == 'primitive' else -0.0252} 0 ${-0.045 if visual_mode == 'primitive' else -0.58444}" rpy="0 0 0"/>
     </collision>
     <inertial>
@@ -45,14 +57,24 @@
     <visual>
         <geometry>
-        <mesh filename="package://caramelo_description/meshes/manipulator/right_finger.stl" scale="0.001 0.001 0.001"/>
+        <xacro:if value="${visual_mode == 'primitive'}">
+        <box size="0.018 0.018 0.090"/>
+        </xacro:if>
+        <xacro:if value="${visual_mode != 'primitive'}">
+        <mesh filename="${mesh_uri_prefix}/meshes/manipulator/right_finger.stl" scale="0.001 0.001 0.001"/>
+        </xacro:if>
         </geometry>
-        <origin xyz="0.0252 0 -0.58444" rpy="0 0 0"/>
+        <origin xyz="${0 if visual_mode == 'primitive' else 0.0252} 0 ${-0.045 if visual_mode == 'primitive' else -0.58444}" rpy="0 0 0"/>
         <material name="grey"/>
     </visual>
     <collision>
         <geometry>
-        <mesh filename="package://caramelo_description/meshes/manipulator/right_finger.stl" scale="0.001 0.001 0.001"/>
+        <xacro:if value="${visual_mode == 'primitive'}">
+        <box size="0.018 0.018 0.090"/>
+        </xacro:if>
+        <xacro:if value="${visual_mode != 'primitive'}">
+        <mesh filename="${mesh_uri_prefix}/meshes/manipulator/right_finger.stl" scale="0.001 0.001 0.001"/>
+        </xacro:if>
         </geometry>
-        <origin xyz="0.0252 0 -0.58444" rpy="0 0 0"/>
+        <origin xyz="${0 if visual_mode == 'primitive' else 0.0252} 0 ${-0.045 if visual_mode == 'primitive' else -0.58444}" rpy="0 0 0"/>
     </collision>
     <inertial>

File: src/caramelo_description/urdf/mech/mecanum_wheel.xacro (robot description, xacro)
@@ -9,20 +9,42 @@
         x_reflect
         y_reflect
+        visual_mode:='package'
         wheel_mesh:='${mecanum_wheel_mesh}'
         wheel_mesh_scale:='${mecanum_wheel_mesh_scale}'">
         <link name="${prefix}${side}_wheel_link">
-            <visual>
-                <origin xyz="0 0 0" rpy="${M_PI/2 if x_reflect == y_reflect else -M_PI/2} 0 0"/>
-                <geometry>
-                    <mesh filename="${wheel_mesh}" scale="${wheel_mesh_scale}"/>
-                </geometry>
-                <material name="orange"/>
-            </visual>
-            <collision>
-                <origin xyz="0 0 0" rpy="${M_PI/2 if x_reflect == y_reflect else -M_PI/2} 0 0"/>
-                <geometry>
-                    <mesh filename="${wheel_mesh}" scale="${wheel_mesh_scale}"/>
-                </geometry>
-            </collision>
+            <xacro:if value="${visual_mode == 'primitive'}">
+                <visual>
+                    <origin xyz="0 0 0" rpy="${M_PI/2} 0 0"/>
+                    <geometry>
+                        <cylinder radius="${wheel_radius}" length="${wheel_width}"/>
+                    </geometry>
+                    <material name="orange"/>
+                </visual>
+            </xacro:if>
+            <xacro:if value="${visual_mode != 'primitive'}">
+                <visual>
+                    <origin xyz="0 0 0" rpy="${M_PI/2 if x_reflect == y_reflect else -M_PI/2} 0 0"/>
+                    <geometry>
+                        <mesh filename="${wheel_mesh}" scale="${wheel_mesh_scale}"/>
+                    </geometry>
+                    <material name="orange"/>
+                </visual>
+            </xacro:if>
+            <xacro:if value="${visual_mode == 'primitive'}">
+                <collision>
+                    <origin xyz="0 0 0" rpy="${M_PI/2} 0 0"/>
+                    <geometry>
+                        <cylinder radius="${wheel_radius}" length="${wheel_width}"/>
+                    </geometry>
+                </collision>
+            </xacro:if>
+            <xacro:if value="${visual_mode != 'primitive'}">
+                <collision>
+                    <origin xyz="0 0 0" rpy="${M_PI/2 if x_reflect == y_reflect else -M_PI/2} 0 0"/>
+                    <geometry>
+                        <mesh filename="${wheel_mesh}" scale="${wheel_mesh_scale}"/>
+                    </geometry>
+                </collision>
+            </xacro:if>
             <xacro:cylinder_inertia m="${wheel_mass}" r="${wheel_radius}" l="${wheel_width}" o_xyz="0 0 0" o_rpy="${M_PI/2} 0 0"/>
         </link>

File: src/caramelo_description/urdf/mech/mobile_base.xacro (robot description, xacro)
@@ -24,5 +24,5 @@
     <xacro:property name="wheel_base" value="0.472"/>
     <xacro:property name="wheel_center_x" value="0.000"/>
-    <xacro:property name="wheel_z" value="${wheel_radius - base_link_z_from_floor}"/>
+    <xacro:property name="wheel_z" value="${wheel_radius - base_link_z_from_floor +0.001}"/>
     <!-- FRAME_CRITICO: offsets medidos do STL ja com a rotacao de 90 graus aplicada abaixo. -->
     <xacro:property name="base_mesh_stl_center_x" value="0.243517868"/>
@@ -34,30 +34,61 @@
     <xacro:property name="lidar_x" value="${0.265 + base_appendage_x/2.0}"/>
     <xacro:property name="lidar_y" value="0.000"/>
-    <xacro:property name="lidar_z" value="${old_base_link_z_from_floor + 0.030 - base_link_z_from_floor}"/>
+    <xacro:property name="lidar_z" value="${old_base_link_z_from_floor + 0.030 - base_link_z_from_floor - 0.015}"/>
     <xacro:property name="lidar_rpy" value="${M_PI} 0 ${M_PI}"/>
     <!-- FRAME_CRITICO: hardware_bringup publica a IMU como imu_link. -->
     <xacro:property name="imu_x" value="${-0.035 + base_appendage_x/2.0}"/>
     <xacro:property name="imu_y" value="0.000"/>
-    <xacro:property name="imu_z" value="${old_base_link_z_from_floor + 0.090 - base_link_z_from_floor}"/>
+    <xacro:property name="imu_z" value="${old_base_link_z_from_floor + 0.090 - base_link_z_from_floor - 0.015}"/>
     <xacro:property name="imu_rpy" value="0 0 0"/>
     <!-- Base completa: footprint + base_link + 4 rodas mecanum -->
-    <xacro:macro name="mobile_base" params="prefix">
+    <xacro:macro name="mobile_base" params="
+        prefix
+        visual_mode:='package'
+        mesh_uri_prefix:='package://caramelo_description'">
     <link name="${prefix}base_footprint"/>
     <link name="${prefix}base_link">
         <!-- Corpo principal do robo -->
-        <visual>
-            <origin xyz="${base_mesh_xyz}" rpy="${base_mesh_rpy}"/>
-            <geometry>
-                <mesh filename="package://caramelo_description/meshes/robot_3d/montagem_robo_final.stl" scale="0.001 0.001 0.001"/>
-            </geometry>
-            <material name="darkgray"/>
-        </visual>
+        <xacro:if value="${visual_mode == 'primitive'}">
+            <visual>
+                <origin xyz="0 0 0" rpy="0 0 0"/>
+                <geometry>
+                    <box size="${base_width_vertical} ${base_width_horizontal} ${base_height}"/>
+                </geometry>
+                <material name="darkgray"/>
+            </visual>
+            <visual>
+                <origin xyz="${base_width_vertical/2.0 + base_appendage_x/2.0} 0 0" rpy="0 0 0"/>
+                <geometry>
+                    <box size="${base_appendage_x} ${base_width_horizontal*0.70} ${base_height*0.45}"/>
+                </geometry>
+                <material name="darkgray"/>
+            </visual>
+        </xacro:if>
+        <xacro:if value="${visual_mode != 'primitive'}">
+            <visual>
+                <origin xyz="${base_mesh_xyz}" rpy="${base_mesh_rpy}"/>
+                <geometry>
+                    <mesh filename="${mesh_uri_prefix}/meshes/robot_3d/montagem_robo_final.stl" scale="0.001 0.001 0.001"/>
+                </geometry>
+                <material name="darkgray"/>
+            </visual>
+        </xacro:if>
         <!-- Colisao do corpo principal -->
-        <collision>
-            <origin xyz="${base_mesh_xyz}" rpy="${base_mesh_rpy}"/>
-            <geometry>
-                <mesh filename="package://caramelo_description/meshes/robot_3d/montagem_robo_final.stl" scale="0.001 0.001 0.001"/>
-            </geometry>
-        </collision>
+        <xacro:if value="${visual_mode == 'primitive'}">
+            <collision>
+                <origin xyz="0 0 0" rpy="0 0 0"/>
+                <geometry>
+                    <box size="${base_width_vertical} ${base_width_horizontal} ${base_height}"/>
+                </geometry>
+            </collision>
+        </xacro:if>
+        <xacro:if value="${visual_mode != 'primitive'}">
+            <collision>
+                <origin xyz="${base_mesh_xyz}" rpy="${base_mesh_rpy}"/>
+                <geometry>
+                    <mesh filename="${mesh_uri_prefix}/meshes/robot_3d/montagem_robo_final.stl" scale="0.001 0.001 0.001"/>
+                </geometry>
+            </collision>
+        </xacro:if>
         <!-- Inercia aproximada por caixa envolvente da base -->
         <xacro:box_inertia
@@ -80,20 +111,28 @@
         side="front_left"
         x_reflect="1"
-        y_reflect="1"/>
+        y_reflect="1"
+        visual_mode="${visual_mode}"
+        wheel_mesh="${mesh_uri_prefix}/meshes/robot_3d/roda_escala_final.stl"/>
     <xacro:mecanum_wheel
         prefix="${prefix}"
         side="front_right"
         x_reflect="1"
-        y_reflect="-1"/>
+        y_reflect="-1"
+        visual_mode="${visual_mode}"
+        wheel_mesh="${mesh_uri_prefix}/meshes/robot_3d/roda_escala_final.stl"/>
     <xacro:mecanum_wheel
         prefix="${prefix}"
         side="back_left"
         x_reflect="-1"
-        y_reflect="1"/>
+        y_reflect="1"
+        visual_mode="${visual_mode}"
+        wheel_mesh="${mesh_uri_prefix}/meshes/robot_3d/roda_escala_final.stl"/>
     <xacro:mecanum_wheel
         prefix="${prefix}"
         side="back_right"
         x_reflect="-1"
-        y_reflect="-1"/>
+        y_reflect="-1"
+        visual_mode="${visual_mode}"
+        wheel_mesh="${mesh_uri_prefix}/meshes/robot_3d/roda_escala_final.stl"/>
     <!-- Lidar no bico, preso direto na base -->
     <xacro:lidar_sensor
@@ -102,5 +141,7 @@
         frame_id="laser_frame"
         xyz_offset="${lidar_x} ${lidar_y} ${lidar_z}"
-        rpy_offset="${lidar_rpy}"/>
+        rpy_offset="${lidar_rpy}"
+        visual_mode="${visual_mode}"
+        mesh_file="${mesh_uri_prefix}/meshes/rplidar/rplidar_s2.stl"/>
     <!-- IMU presa direto na base -->
     <xacro:imu_sensor

File: src/caramelo_description/urdf/robots/manipulator.urdf.xacro (robot description, xacro)
@@ -3,4 +3,6 @@
   <xacro:arg name="use_realsense" default="true"/>
   <xacro:arg name="use_mock_components" default="true"/>
+  <xacro:arg name="visual_mode" default="package"/>
+  <xacro:arg name="mesh_uri_prefix" default="package://caramelo_description"/>
   <xacro:include filename="../materials.xacro"/>
   <xacro:include filename="../mech/manipulator_arm.xacro"/>
@@ -8,6 +10,12 @@
   <xacro:include filename="../control/manipulator.ros2_control.xacro"/>
   <xacro:manipulator_ros2_control use_mock_components="$(arg use_mock_components)"/>
-  <xacro:manip_arm base_link_name="base_link" use_realsense="$(arg use_realsense)"/>
-  <xacro:manip_gripper/>
+  <xacro:manip_arm
+    base_link_name="base_link"
+    use_realsense="$(arg use_realsense)"
+    visual_mode="$(arg visual_mode)"
+    mesh_uri_prefix="$(arg mesh_uri_prefix)"/>
+  <xacro:manip_gripper
+    visual_mode="$(arg visual_mode)"
+    mesh_uri_prefix="$(arg mesh_uri_prefix)"/>
   <joint name="gripper_base_joint" type="fixed">
     <parent link="link5"/>
