Commit message: Refactor robot description and launch configurations
- Updated mobile_base.xacro to support visual modes and mesh URI prefixes.
- Modified manipulator.urdf.xacro and robot.urdf.xacro to include visual mode and mesh URI arguments.
- Enhanced lidar_sensor.xacro to allow for visual mode selection.
- Adjusted caramelo_controllers.yaml to include arm and gripper controllers with updated parameters.
- Removed obsolete manip_ros2_controllers.yaml and consolidated configurations into caramelo_controllers.yaml.
- Updated rplidar_s2.yaml to change serial port and scan mode.
- Added USB rules for stable device naming on Raspberry Pi.
- Introduced scan_normalizer.yaml and scan_normalizer.py for processing LaserScan messages.
- Cleaned up unused launch files related to manipulator control.
- Added rviz_remote.launch.py for remote RViz configuration.

File: src/caramelo_description/urdf/robots/robot.urdf.xacro (robot description, xacro)
@@ -7,6 +7,8 @@
   <xacro:arg name="use_realsense" default="true"/>
   <xacro:arg name="use_mock_components" default="true"/>
-  <xacro:arg name="manip_mount_xyz" default="0.185 0 0.078"/>
+  <xacro:arg name="manip_mount_xyz" default="0.217 0 0.083"/>
   <xacro:arg name="manip_mount_rpy" default="0 0 0"/>
+  <xacro:arg name="visual_mode" default="package"/>
+  <xacro:arg name="mesh_uri_prefix" default="package://caramelo_description"/>
   <!-- Includes -->
   <xacro:include filename="../materials.xacro"/>
@@ -16,5 +18,8 @@
   <xacro:include filename="../mech/caramelo_manipulator.xacro"/>
   <!-- Base movel completa (base_link + footprint + 4 rodas) -->
-  <xacro:mobile_base prefix="$(arg prefix)"/>
+  <xacro:mobile_base
+    prefix="$(arg prefix)"
+    visual_mode="$(arg visual_mode)"
+    mesh_uri_prefix="$(arg mesh_uri_prefix)"/>
   <xacro:if value="$(arg use_manipulator)">
     <xacro:caramelo_manipulator
@@ -23,5 +28,7 @@
       use_realsense="$(arg use_realsense)"
       manip_mount_xyz="$(arg manip_mount_xyz)"
-      manip_mount_rpy="$(arg manip_mount_rpy)"/>
+      manip_mount_rpy="$(arg manip_mount_rpy)"
+      visual_mode="$(arg visual_mode)"
+      mesh_uri_prefix="$(arg mesh_uri_prefix)"/>
     <xacro:manipulator_ros2_control use_mock_components="$(arg use_mock_components)"/>
   </xacro:if>

File: src/caramelo_description/urdf/sensors/lidar_sensor.xacro (robot description, xacro)
@@ -6,4 +6,5 @@
     parent:='base_link'
     frame_id:='laser_frame'
+    visual_mode:='package'
     mesh_file:='package://caramelo_description/meshes/rplidar/rplidar_s2.stl'
     xyz_offset:='0 0 0.0825'
@@ -39,19 +40,40 @@
     <xacro:property name="izz" value="${(mass/2) * (radius * radius)}" />
     <link name="${prefix}${frame_id}">
-      <visual>
-        <origin xyz="${mesh_xyz_offset}" rpy="${mesh_rpy_offset}"/>
-        <geometry>
-          <mesh filename="${mesh_file}" scale="${mesh_scale}"/>
-        </geometry>
-        <material name="${material_name}">
-          <color rgba="${material_color}"/>
-        </material>
-      </visual>
-      <xacro:if value="${enable_collision}">
-        <collision>
+      <xacro:if value="${visual_mode == 'primitive'}">
+        <visual>
+          <origin xyz="0 0 0" rpy="0 0 0"/>
+          <geometry>
+            <cylinder radius="${radius}" length="${lidar_height}"/>
+          </geometry>
+          <material name="${material_name}">
+            <color rgba="${material_color}"/>
+          </material>
+        </visual>
+      </xacro:if>
+      <xacro:if value="${visual_mode != 'primitive'}">
+        <visual>
           <origin xyz="${mesh_xyz_offset}" rpy="${mesh_rpy_offset}"/>
           <geometry>
             <mesh filename="${mesh_file}" scale="${mesh_scale}"/>
           </geometry>
+          <material name="${material_name}">
+            <color rgba="${material_color}"/>
+          </material>
+        </visual>
+      </xacro:if>
+      <xacro:if value="${enable_collision}">
+        <collision>
+          <xacro:if value="${visual_mode == 'primitive'}">
+            <origin xyz="0 0 0" rpy="0 0 0"/>
+            <geometry>
+              <cylinder radius="${radius}" length="${lidar_height}"/>
+            </geometry>
+          </xacro:if>
+          <xacro:if value="${visual_mode != 'primitive'}">
+            <origin xyz="${mesh_xyz_offset}" rpy="${mesh_rpy_offset}"/>
+            <geometry>
+              <mesh filename="${mesh_file}" scale="${mesh_scale}"/>
+            </geometry>
+          </xacro:if>
         </collision>
       </xacro:if>
