Commit message: hardware bringup correction

File: src/caramelo_description/urdf/control/mobile_base.ros2_control.xacro (robot description, xacro)
@@ -3,9 +3,12 @@
     <ros2_control name="MobileBaseHardwareInterface" type="system">
         <hardware>
-            <!--* Qual o plugin de hardware a ser utilizado? -->
-            <!--* Mock components: Somente para simulação -->
-            <!-- <plugin>mock_components/GenericSystem</plugin> -->
-            <!--* Mobile base hardware interface: Para controle real do robô -->
-            <plugin>mobile_base_hardware/MobileBaseHWInterface</plugin>
+            <xacro:if value="$(arg use_mock_components)">
+                <!--* Mock components: Somente para validação sem hardware real -->
+                <plugin>mock_components/GenericSystem</plugin>
+            </xacro:if>
+            <xacro:unless value="$(arg use_mock_components)">
+                <!--* Mobile base hardware interface: Para controle real do robô -->
+                <plugin>mobile_base_hardware/MobileBaseHWInterface</plugin>
+            </xacro:unless>
         </hardware>
         <!-- Criar uma joint tag para cada junta que desejar que seja controlada -->

File: src/caramelo_description/urdf/robots/robot.urdf.xacro (robot description, xacro)
@@ -8,5 +8,5 @@
   <xacro:arg name="use_mock_components" default="true"/>
   <xacro:arg name="manip_mount_xyz" default="0.217 0 0.083"/>
-  <xacro:arg name="manip_mount_rpy" default="0 0 0"/>
+  <xacro:arg name="manip_mount_rpy" default="0 0 -1.57"/>
   <xacro:arg name="visual_mode" default="package"/>
   <xacro:arg name="mesh_uri_prefix" default="package://caramelo_description"/>

File: src/caramelo_description/urdf/sensors/realsense/_d455.urdf.xacro (robot description, xacro)
@@ -23,5 +23,11 @@
   <xacro:include filename="$(find caramelo_description)/urdf/sensors/realsense/_materials.urdf.xacro" />
   <xacro:include filename="$(find caramelo_description)/urdf/sensors/realsense/_usb_plug.urdf.xacro" />
-  <xacro:macro name="sensor_d455" params="parent *origin name:=camera use_nominal_extrinsics:=false">
+  <xacro:macro name="sensor_d455" params="
+    parent
+    *origin
+    name:=camera
+    use_nominal_extrinsics:=false
+    visual_mode:='package'
+    mesh_uri_prefix:='package://caramelo_description'">
     <xacro:arg name="add_plug" default="false" />
     <xacro:property name="M_PI" value="3.1415926535897931" />
@@ -67,6 +73,10 @@
         <origin xyz="${d455_zero_depth_to_glass + d455_glass_to_front} ${-d455_cam_depth_py} 0" rpy="${M_PI/2} 0 ${M_PI/2}"/>
         <geometry>
-          <!-- <box size="${d455_cam_depth} ${d455_cam_width} ${d455_cam_height}"/> -->
-          <mesh filename="package://caramelo_description/meshes/intel_realsense/d455.stl" scale="0.001 0.001 0.001" />
+          <xacro:if value="${visual_mode == 'primitive'}">
+            <box size="${d455_cam_depth} ${d455_cam_width} ${d455_cam_height}"/>
+          </xacro:if>
+          <xacro:if value="${visual_mode != 'primitive'}">
+            <mesh filename="${mesh_uri_prefix}/meshes/intel_realsense/d455.stl" scale="0.001 0.001 0.001" />
+          </xacro:if>
         </geometry>
         <material name="aluminum"/>
@@ -176,5 +186,9 @@
     </xacro:if>
     <xacro:if value="$(arg add_plug)">
-      <xacro:usb_plug parent="${name}_link" name="${name}_usb_plug">
+      <xacro:usb_plug
+          parent="${name}_link"
+          name="${name}_usb_plug"
+          visual_mode="${visual_mode}"
+          mesh_uri_prefix="${mesh_uri_prefix}">
         <origin xyz="${-0.00406-d455_cam_depth_px} ${-0.03701-d455_cam_depth_py} ${-d455_cam_depth_pz}" rpy="${M_PI/2} 0 0"/>
       </xacro:usb_plug>

File: src/caramelo_description/urdf/sensors/realsense/_usb_plug.urdf.xacro (robot description, xacro)
@@ -20,5 +20,10 @@
 -->
 <robot name="usb_plug" xmlns:xacro="http://ros.org/wiki/xacro">
-  <xacro:macro name="usb_plug" params="parent *origin name:=usb_plug">
+  <xacro:macro name="usb_plug" params="
+    parent
+    *origin
+    name:=usb_plug
+    visual_mode:='package'
+    mesh_uri_prefix:='package://caramelo_description'">
     <xacro:property name="M_PI" value="3.1415926535897931" />
     <joint name="${name}_joint" type="fixed">
@@ -32,6 +37,10 @@
         <origin xyz="0. -0.022425 0." rpy="0 0 ${M_PI/2}"/>
         <geometry>
-          <!--box size="0.044850 0.008 0.0185" /-->
-          <mesh filename="package://caramelo_description/meshes/intel_realsense/plug.stl" />
+          <xacro:if value="${visual_mode == 'primitive'}">
+            <box size="0.044850 0.008 0.0185"/>
+          </xacro:if>
+          <xacro:if value="${visual_mode != 'primitive'}">
+            <mesh filename="${mesh_uri_prefix}/meshes/intel_realsense/plug.stl" />
+          </xacro:if>
         </geometry>
         <material name="plastic"/>
@@ -40,6 +49,10 @@
         <origin xyz="0. -0.022425 0." rpy="0 0 ${M_PI/2}"/>
         <geometry>
-          <!--box size="0.044850 0.008 0.0185" /-->
-          <mesh filename="package://caramelo_description/meshes/intel_realsense/plug_collision.stl" />
+          <xacro:if value="${visual_mode == 'primitive'}">
+            <box size="0.044850 0.008 0.0185"/>
+          </xacro:if>
+          <xacro:if value="${visual_mode != 'primitive'}">
+            <mesh filename="${mesh_uri_prefix}/meshes/intel_realsense/plug_collision.stl" />
+          </xacro:if>
         </geometry>
       </collision>

File: src/caramelo_description/urdf/sensors/rgbd_camera.urdf.xacro (robot description, xacro)
@@ -6,5 +6,7 @@
     xyz_offset:='0 0 0'
     rpy_offset:='0 0 0'
-    use_nominal_extrinsics:=true">
+    use_nominal_extrinsics:=true
+    visual_mode:='package'
+    mesh_uri_prefix:='package://caramelo_description'">
     <!-- Intel RealSense D455 vendorizada no caramelo_description. -->
     <xacro:include filename="$(find caramelo_description)/urdf/sensors/realsense/_d455.urdf.xacro"/>
@@ -12,5 +14,7 @@
         parent="${parent}"
         name="${camera_name}"
-        use_nominal_extrinsics="${use_nominal_extrinsics}">
+        use_nominal_extrinsics="${use_nominal_extrinsics}"
+        visual_mode="${visual_mode}"
+        mesh_uri_prefix="${mesh_uri_prefix}">
       <origin xyz="${xyz_offset}" rpy="${rpy_offset}"/>
     </xacro:sensor_d455>
